Commit message: Enhance ROMI simulation support with updated launch files and Gazebo integration; refactor URDF and RViz configurations

File: romi_base/description/urdf/romi.urdf.xacro (robot description, xacro)
@@ -6,21 +6,22 @@
     <!-- <xacro:include filename="romi_camera.xacro"/> -->
     <xacro:include filename="romi_lidar.xacro"/>
-    <!-- For sim only: drive the wheel joints from /cmd_vel in Gazebo. -->
+    <!-- For sim only: drive wheel joints and publish odom/joint states. -->
     <xacro:if value="$(arg use_simulation)">
         <gazebo>
-            <plugin name="diff_drive_controller" filename="libgazebo_ros_diff_drive.so">
-                <ros>
-                    <remapping>cmd_vel:=/cmd_vel</remapping>
-                    <remapping>odom:=/odom</remapping>
-                </ros>
-                <update_rate>50</update_rate>
+            <plugin filename="ignition-gazebo6-diff-drive-system" name="ignition::gazebo::systems::DiffDrive">
                 <left_joint>left_wheel_joint</left_joint>
                 <right_joint>right_wheel_joint</right_joint>
                 <wheel_separation>0.141</wheel_separation>
                 <wheel_radius>0.035</wheel_radius>
-                <publish_odom>true</publish_odom>
-                <publish_odom_tf>true</publish_odom_tf>
-                <odometry_frame>odom</odometry_frame>
-                <robot_base_frame>base_link</robot_base_frame>
+                <topic>/cmd_vel</topic>
+                <odom_topic>/odom</odom_topic>
+                <tf_topic>/tf</tf_topic>
+                <frame_id>odom</frame_id>
+                <child_frame_id>base_link</child_frame_id>
+            </plugin>
+            <plugin filename="ignition-gazebo6-joint-state-publisher-system" name="ignition::gazebo::systems::JointStatePublisher">
+                <topic>/joint_states</topic>
+                <joint_name>left_wheel_joint</joint_name>
+                <joint_name>right_wheel_joint</joint_name>
             </plugin>
         </gazebo>

File: romi_base/description/urdf/romi_core.xacro (robot description, xacro)
@@ -48,12 +48,12 @@
             <origin xyz="${chassis_length/2} 0 0"/>
             <geometry>
-                <mesh filename="package://romi_base/description/meshes/romi_chassis_low.stl" scale="1 1 1"/>
+                <mesh filename="file://$(find romi_base)/description/meshes/romi_chassis.stl" scale="1 1 1"/>
             </geometry>
             <material name="orange"/>
         </visual>
         <collision>
-            <origin xyz="${chassis_length/2} 0 0"/>
+            <origin xyz="${chassis_length/2} 0 ${chassis_height/2}"/>
             <geometry>
-                <mesh filename="package://romi_base/description/meshes/romi_chassis_low.stl" scale="1 1 1"/>
+                <box size="${chassis_length} ${chassis_width} ${chassis_height}"/>
             </geometry>
         </collision>
@@ -77,5 +77,5 @@
         <visual>
             <geometry>
-                <mesh filename="package://romi_base/description/meshes/left_wheel2.stl" scale="1 1 1"/>
+                <mesh filename="file://$(find romi_base)/description/meshes/left_wheel2.stl" scale="1 1 1"/>
             </geometry>
             <material name="blue"/>
@@ -83,5 +83,5 @@
         <collision>
             <geometry>
-                <mesh filename="package://romi_base/description/meshes/left_wheel2.stl" scale="1 1 1"/>
+                <cylinder radius="${wheel_radius}" length="${wheel_thickness}"/>
             </geometry>
         </collision>
@@ -103,5 +103,5 @@
         <visual>
             <geometry>
-                <mesh filename="package://romi_base/description/meshes/right_wheel2.stl" scale="1 1 1"/>
+                <mesh filename="file://$(find romi_base)/description/meshes/right_wheel2.stl" scale="1 1 1"/>
             </geometry>
             <material name="blue"/>
@@ -109,5 +109,5 @@
         <collision>
             <geometry>
-                <mesh filename="package://romi_base/description/meshes/right_wheel2.stl" scale="1 1 1"/>
+                <cylinder radius="${wheel_radius}" length="${wheel_thickness}"/>
             </geometry>
         </collision>

File: romi_base/description/urdf/romi_lidar.xacro (robot description, xacro)
@@ -18,6 +18,8 @@
         <sensor name="laser" type="ray">
             <pose> 0 0 0 0 0 0 </pose>
+            <always_on>true</always_on>
             <visualize>true</visualize>
             <update_rate>10</update_rate>
+            <topic>/scan</topic>
             <ray>
                 <scan>
@@ -33,11 +35,4 @@
                 </range>
             </ray>
-            <plugin name="laser_controller" filename="libgazebo_ros_ray_sensor.so">
-                <ros>
-                    <remapping>~/out:=/scan</remapping>
-                </ros>
-                <output_type>sensor_msgs/LaserScan</output_type>
-                <frame_name>lidar_frame</frame_name>
-            </plugin>
         </sensor>
     </gazebo>
