Commit message: Update launch files and scripts for improved configuration and functionality
- Change default frame ID from 'laser' to 'lidar_frame' in romi_robot.launch.py and rplidar_a1_launch.py for consistency.
- Modify mesh file paths in romi_core.xacro to use 'package://' syntax for better compatibility.
- Add postStartCommand in devcontainer.json to ensure ROS environment is sourced in .bashrc.
- Enhance sync_to_pi.sh script to include a --clean option for optional removal of remote build artifacts before syncing.

File: romi_base/description/urdf/romi_core.xacro (robot description, xacro)
@@ -48,7 +48,7 @@
             <origin xyz="${chassis_length/2} 0 0"/>
             <geometry>
-                <mesh filename="file://$(find romi_base)/description/meshes/romi_chassis.stl" scale="1 1 1"/>
+                <mesh filename="package://romi_base/description/meshes/romi_chassis.stl" scale="1 1 1"/>
             </geometry>
-            <material name="orange"/>
+            <material name="blue"/>
         </visual>
         <collision>
@@ -77,5 +77,5 @@
         <visual>
             <geometry>
-                <mesh filename="file://$(find romi_base)/description/meshes/left_wheel2.stl" scale="1 1 1"/>
+                <mesh filename="package://romi_base/description/meshes/left_wheel2.stl" scale="1 1 1"/>
             </geometry>
             <material name="blue"/>
@@ -103,5 +103,5 @@
         <visual>
             <geometry>
-                <mesh filename="file://$(find romi_base)/description/meshes/right_wheel2.stl" scale="1 1 1"/>
+                <mesh filename="package://romi_base/description/meshes/right_wheel2.stl" scale="1 1 1"/>
             </geometry>
             <material name="blue"/>
