Commit message: Fixed lidar xacro problem

File: romi_base/description/urdf/romi_lidar.xacro (robot description, xacro)
@@ -4,5 +4,5 @@
         <parent link="chassis"/>
         <child link="lidar_frame"/>
-        <origin xyz="${chassis_length/2} 0 0.105" rpy="${pi} 0 0"/>
+        <origin xyz="${chassis_length/2} 0 0.105" rpy="0 0 0"/>
     </joint>
     <link name="lidar_frame">
