Commit message: Refactor ROMI base controller and launch files
- Updated the base_controller_node.py to improve code structure and readability, including changes to the PI controller implementation and odometry calculations.
- Removed the romi_rviz_only.launch.py file and integrated its functionality into existing launch files.
- Modified URDF files to use the correct mesh file paths and changed the material color for the chassis.
- Updated launch files to include joint_state_publisher as an optional argument for better visualization in RViz.
- Changed the lidar sensor type from gpu_lidar to ray in the romi_lidar.xacro file for compatibility with Ignition Gazebo.
- Adjusted the launch configurations for Gazebo to support GUI options and improved the handling of simulation parameters.

File: install/romi_base/share/romi_base/description/urdf/romi_core.xacro (robot description, xacro)
@@ -48,7 +48,7 @@
             <origin xyz="${chassis_length/2} 0 0"/>
             <geometry>
-                <mesh filename="package://romi_base/description/meshes/romi_chassis.stl" scale="1 1 1"/>
+                <mesh filename="file://$(find romi_base)/description/meshes/romi_chassis.stl" scale="1 1 1"/>
             </geometry>
-            <material name="blue"/>
+            <material name="orange"/>
         </visual>
         <collision>
@@ -77,5 +77,5 @@
         <visual>
             <geometry>
-                <mesh filename="package://romi_base/description/meshes/left_wheel2.stl" scale="1 1 1"/>
+                <mesh filename="file://$(find romi_base)/description/meshes/left_wheel2.stl" scale="1 1 1"/>
             </geometry>
             <material name="blue"/>
@@ -103,5 +103,5 @@
         <visual>
             <geometry>
-                <mesh filename="package://romi_base/description/meshes/right_wheel2.stl" scale="1 1 1"/>
+                <mesh filename="file://$(find romi_base)/description/meshes/right_wheel2.stl" scale="1 1 1"/>
             </geometry>
             <material name="blue"/>
